File: hardware/pc_fdc1004_brk_v3.sch (EAGLE design)
At the start: 19 parts, among them Q1 BSS138, Q2 BSS138

Commit message: schematics,images and readme updated
Parts:
- removed C69: 10n, rcl:C-EUC0805
- removed C70, C74: 1u, rcl:C-EUC0805
- removed R10: 0R, rcl:R-US_R0805
- removed U$27: TPS71733, circuitects:TPS717XX
- removed U$6: PROTY_LOGO_WITH_TEXT, circuitects:PROTY_LOGO_WITH_TEXT
- added C11: 1u, rcl:C-EUC0402
- added C24: 2.2uF, rcl:C-EUC0402
- added J1, J2: Qwiic1, SparkFun-Connectors:QWIIC_CONNECTORJS-1MM
- added U2: AP2112K-3.3V, SparkFun-PowerIC:V_REG_LDOSMD
Connections:
- removed net N$2: C74.2, R10.2, U$27.EN, U$27.IN
- removed net N$70: C69.2, U$27.FB
- net +3V3: now also C24.1, J1.2, J2.2, U2.OUT; no longer C70.2, U$27.OUT
- net FDC_SCL: now also J1.4, J2.4
- net FDC_SDA: now also J1.3, J2.3
- net GND: now also C11.1, C24.2, J1.1, J2.1, U2.GND; no longer C69.1, C70.1, C74.1, U$27.GND
- net VCC: now also C11.2, U2.EN, U2.IN; no longer R10.1
